File: ti92revive/ti92revive.kicad_pcb (KiCad board)
At the start: 2 copper layers, 205 x 113.6 mm, 0 parts

Commit message: Add files via upload
Parts:
- added IC1: TCA8418, 18650:TCA8418-WQFN-24-1EP_4x4mm, B.Cu at (138.2, 87.4)
- added R1: 4.7k, Resistor_SMD:R_0805_2012Metric_Pad1.15x1.40mm_HandSolder, F.Cu at (135.0, 101.6)
- added R2: 10k, Resistor_SMD:R_0805_2012Metric_Pad1.15x1.40mm_HandSolder, F.Cu at (138.9, 101.6)
- added REF**: LOGOMORH, 18650:LOGOMORH, F.Cu at (138.9, 79.0)
- added arrwDWN1: ArwDwn, 18650:Kbpad, F.Cu at (235.3, 69.5)
- added arrwLeft1: ArwLeft, 18650:Kbpad, F.Cu at (226.3, 60.3)
- added arrwRight1: ArwRight, 18650:Kbpad, F.Cu at (244.5, 60.3)
- added arrwUP1: ArwUP, 18650:Kbpad, F.Cu at (235.3, 51.4)
- added kN666: 6, 18650:Kbpad, F.Cu at (229.9, 120.8)
- added kb2nd1: 2ndUP, 18650:Kbpad, F.Cu at (204.1, 48.5)
- added kbA1: A, 18650:Kbpad, F.Cu at (74.5, 120.7)
- added kbALT1: Alt, 18650:Kbpad, F.Cu at (81.2, 141.1)
- added kbALTG1: AltG, 18650:Kbpad, F.Cu at (160.8, 141.1)
- added kbAPPS1: Apps, 18650:Kbpad, F.Cu at (216.9, 69.8)
- added kbAPPS2: Apps, 18650:Kbpad, F.Cu at (217.0, 80.0)
- added kbAnex2: BTN2, 18650:Kbpad, F.Cu at (94.5, 141.0)
- added kbB1: B, 18650:Kbpad, F.Cu at (134.1, 130.8)
- added kbBKSP1: BckSp, 18650:Kbpad, F.Cu at (173.9, 141.0)
- added kbC1: C, 18650:Kbpad, F.Cu at (107.6, 130.8)
- added kbCOS1: Cos, 18650:Kbpad, F.Cu at (217.0, 90.2)
- added kbCTRL1: CTRL, 18650:Kbpad, F.Cu at (67.9, 141.1)
- added kbClear1: Clear, 18650:Kbpad, F.Cu at (204.1, 70.0)
- added kbComa1: Coma, 18650:Kbpad, F.Cu at (230.0, 100.5)
- added kbD1: D, 18650:Kbpad, F.Cu at (101.1, 120.7)
- added kbDiv1: /, 18650:Kbpad, F.Cu at (242.6, 100.5)
- added kbDot1: ., 18650:Kbpad, F.Cu at (217.2, 141.0)
- added kbDot2: Tet, 18650:Kbpad, F.Cu at (174.0, 130.8)
- added kbENT1: ENTER, 18650:Kbpad, F.Cu at (242.7, 142.0)
- added kbESC1: ESC, 18650:Kbpad, F.Cu at (218.3, 48.4)
- added kbESC55: ESC, 18650:Kbpad, F.Cu at (215.4, 59.1)
- added kbEnterNum1: EnterN, 18650:Kbpad, F.Cu at (230.1, 80.0)
- added kbEnterNum66: EnterN, 18650:Kbpad, F.Cu at (241.9, 80.0)
- added kbF1: F, 18650:Kbpad, F.Cu at (114.2, 120.7)
- added kbG1: G, 18650:Kbpad, F.Cu at (127.5, 120.7)
- added kbH1: H, 18650:Kbpad, F.Cu at (140.7, 120.7)
- added kbI1: I, 18650:Kbpad, F.Cu at (160.7, 110.6)
- added kbJ1: J, 18650:Kbpad, F.Cu at (154.1, 120.7)
- added kbK1: K, 18650:Kbpad, F.Cu at (167.3, 120.7)
- added kbL1: L, 18650:Kbpad, F.Cu at (180.5, 120.7)
- added kbLBrack1: (, 18650:Kbpad, F.Cu at (204.3, 100.5)
- added kbLn1: LN, 18650:Kbpad, F.Cu at (204.2, 80.0)
- added kbM1: M, 18650:Kbpad, F.Cu at (160.8, 130.8)
- added kbMinus1: Minus, 18650:Kbpad, F.Cu at (242.7, 120.7)
- added kbMode1: Mode, 18650:Kbpad, F.Cu at (204.1, 59.4)
- added kbMult1: *, 18650:Kbpad, F.Cu at (242.6, 110.5)
- added kbN1: 1, 18650:Kbpad, F.Cu at (204.3, 130.8)
- added kbN2: 2, 18650:Kbpad, F.Cu at (217.2, 130.7)
- added kbN3: 3, 18650:Kbpad, F.Cu at (229.9, 130.7)
- added kbN4: 0, 18650:Kbpad, F.Cu at (204.3, 141.0)
- added kbN5: 7, 18650:Kbpad, F.Cu at (204.2, 110.5)
- added kbN521: 5, 18650:Kbpad, F.Cu at (217.0, 120.8)
- added kbN6: N, 18650:Kbpad, F.Cu at (147.3, 130.8)
- added kbN7: 8, 18650:Kbpad, F.Cu at (217.2, 110.5)
- added kbN8: 9, 18650:Kbpad, F.Cu at (229.9, 110.5)
- added kbN9: 4, 18650:Kbpad, F.Cu at (204.3, 120.8)
- added kbNeg1: (-), 18650:Kbpad, F.Cu at (230.0, 141.0)
- added kbO1: O, 18650:Kbpad, F.Cu at (173.7, 110.6)
- added kbP1: P, 18650:Kbpad, F.Cu at (187.1, 110.6)
- added kbPI1: PI, 18650:Kbpad, F.Cu at (242.7, 90.0)
- added kbPLUS1: +, 18650:Kbpad, F.Cu at (242.6, 130.7)
- added kbQ1: Q, 18650:Kbpad, F.Cu at (67.8, 110.6)
- added kbR1: R, 18650:Kbpad, F.Cu at (107.6, 110.6)
- added kbRBrack1: ), 18650:Kbpad, F.Cu at (217.2, 100.5)
- added kbRET1: Return, 18650:Kbpad, F.Cu at (187.2, 130.8)
- added kbRET32: Return, 18650:Kbpad, F.Cu at (187.2, 141.0)
- added kbS1: S, 18650:Kbpad, F.Cu at (87.9, 120.7)
- added kbSIN1: Sin, 18650:Kbpad, F.Cu at (204.2, 90.2)
- added kbShiftL1: L-Shift, 18650:Kbpad, F.Cu at (67.9, 130.8)
- added kbSpace1: Space, 18650:Kbpad, F.Cu at (124.2, 141.1)
- added kbSpace2: Space, 18650:Kbpad, F.Cu at (144.1, 141.1)
- added kbT1: T, 18650:Kbpad, F.Cu at (120.8, 110.6)
- added kbTAB1: TAB, 18650:Kbpad, F.Cu at (107.6, 141.0)
- added kbTAN1: Tan, 18650:Kbpad, F.Cu at (229.9, 90.2)
- added kbU1: U, 18650:Kbpad, F.Cu at (147.3, 110.6)
- added kbV1: V, 18650:Kbpad, F.Cu at (120.8, 130.8)
- added kbW1: W, 18650:Kbpad, F.Cu at (81.2, 110.6)
- added kbX1: X, 18650:Kbpad, F.Cu at (94.5, 130.8)
- added kbY1: Y, 18650:Kbpad, F.Cu at (134.1, 110.6)
- added kbZ1: Z, 18650:Kbpad, F.Cu at (81.0, 130.8)
- added kf1: F1, 18650:Kbpad, F.Cu at (67.8, 62.6)
- added kf2: F2, 18650:Kbpad, F.Cu at (67.8, 73.3)
- added kf3: F3, 18650:Kbpad, F.Cu at (67.9, 83.8)
- added kf4: F4, 18650:Kbpad, F.Cu at (67.9, 94.4)
- added kf5: F5, 18650:Kbpad, F.Cu at (81.0, 62.5)
- added kf6: F6, 18650:Kbpad, F.Cu at (81.2, 73.3)
- added kf7: F7, 18650:Kbpad, F.Cu at (81.0, 83.7)
- added kf8: F8, 18650:Kbpad, F.Cu at (81.2, 94.4)
- added klock1: lock, 18650:Kbpad, F.Cu at (80.9, 49.8)
- added kwE1: E, 18650:Kbpad, F.Cu at (94.5, 110.6)
Other:
- net class Default removed
